File: lab4/Exercise 1/Exercise 1.kicad_sch (KiCad schematic)
At the start: 6 parts, among them SW1 SW_SPDT

Commit message: added lab6
Parts:
- C1: footprint (none) -> Capacitor_THT:C_Radial_D5.0mm_H5.0mm_P2.00mm
- D1: footprint (none) -> LED_THT:LED_D5.0mm
- R1, R2: footprint (none) -> Resistor_THT:R_Axial_DIN0516_L15.5mm_D5.0mm_P20.32mm_Horizontal
- SW1: footprint (none) -> Button_Switch_THT:SW_E-Switch_EG1224_SPDT_Angled
- V1: footprint (none) -> Connector_JST:JST_PH_B2B-PH-K_1x02_P2.00mm_Vertical
Changed lines of the file:
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@@
       (effects (font (size 1.27 1.27)) (justify right))
     )
-    (property "Footprint" "" (id 2) (at 133.35 82.55 0)
+    (property "Footprint" "LED_THT:LED_D5.0mm" (id 2) (at 133.35 82.55 0)
       (effects (font (size 1.27 1.27)) hide)
     )
@@
     (property "Reference" "R1" (id 0) (at 138.43 68.58 90))
     (property "Value" "20k Ω" (id 1) (at 135.89 68.58 90))
-    (property "Footprint" "" (id 2) (at 135.128 68.58 90)
+    (property "Footprint" "Resistor_THT:R_Axial_DIN0516_L15.5mm_D5.0mm_P20.32mm_Horizontal" (id 2) (at 135.128 68.58 90)
       (effects (font (size 1.27 1.27)) hide)
     )
@@
   )
   (symbol (lib_id "Device:R") (at 82.55 62.23 90) (unit 1)
-    (in_bom yes) (on_board yes) (fields_autoplaced)
+    (in_bom yes) (on_board yes)
     (property "Reference" "R2" (id 0) (at 82.55 55.88 90))
     (property "Value" "2.2k Ω" (id 1) (at 82.55 58.42 90))
-    (property "Footprint" "" (id 2) (at 82.55 64.008 90)
+    (property "Footprint" "Resistor_THT:R_Axial_DIN0516_L15.5mm_D5.0mm_P20.32mm_Horizontal" (id 2) (at 69.85 43.18 90)
       (effects (font (size 1.27 1.27)) hide)
     )
@@
       (effects (font (size 1.27 1.27)) (justify left))
     )
-    (property "Footprint" "" (id 2) (at 113.9952 74.93 0)
+    (property "Footprint" "Capacitor_THT:C_Radial_D5.0mm_H5.0mm_P2.00mm" (id 2) (at 113.9952 74.93 0)
       (effects (font (size 1.27 1.27)) hide)
     )
@@
     (property "Reference" "SW1" (id 0) (at 99.06 54.61 0))
     (property "Value" "SW_SPDT" (id 1) (at 99.06 57.15 0))
-    (property "Footprint" "" (id 2) (at 99.06 62.23 0)
+    (property "Footprint" "Button_Switch_THT:SW_E-Switch_EG1224_SPDT_Angled" (id 2) (at 99.06 62.23 0)
       (effects (font (size 1.27 1.27)) hide)
     )
@@
   )
   (symbol (lib_id "Connector:Conn_01x02_Male") (at 64.77 74.93 0) (unit 1)
-    (in_bom yes) (on_board yes) (fields_autoplaced)
+    (in_bom yes) (on_board yes)
     (property "Reference" "V1" (id 0) (at 65.405 69.85 0))
     (property "Value" "9V" (id 1) (at 65.405 72.39 0))
-    (property "Footprint" "" (id 2) (at 64.77 74.93 0)
+    (property "Footprint" "Connector_JST:JST_PH_B2B-PH-K_1x02_P2.00mm_Vertical" (id 2) (at 40.64 90.17 0)
       (effects (font (size 1.27 1.27)) hide)
     )
@@
   (symbol_instances
     (path "/7c217758-5787-43ee-8797-0ebdd7082414"
-      (reference "C1") (unit 1) (value "4.7 µF") (footprint "")
+      (reference "C1") (unit 1) (value "4.7 µF") (footprint "Capacitor_THT:C_Radial_D5.0mm_H5.0mm_P2.00mm")
     )
     (path "/42049f09-0cc7-48cb-881c-c12e4c4ffd8a"
-      (reference "D1") (unit 1) (value "LED") (footprint "")
+      (reference "D1") (unit 1) (value "LED") (footprint "LED_THT:LED_D5.0mm")
     )
     (path "/57ace551-3cbb-4ced-ac02-dc6a05a84267"
-      (reference "R1") (unit 1) (value "20k Ω") (footprint "")
+      (reference "R1") (unit 1) (value "20k Ω") (footprint "Resistor_THT:R_Axial_DIN0516_L15.5mm_D5.0mm_P20.32mm_Horizontal")
     )
     (path "/5aca882b-c512-40f0-bf1e-835ac504557d"
-      (reference "R2") (unit 1) (value "2.2k Ω") (footprint "")
+      (reference "R2") (unit 1) (value "2.2k Ω") (footprint "Resistor_THT:R_Axial_DIN0516_L15.5mm_D5.0mm_P20.32mm_Horizontal")
     )
     (path "/7e686513-e7a6-4c64-a3da-0fdbccfb4eeb"
-      (reference "SW1") (unit 1) (value "SW_SPDT") (footprint "")
+      (reference "SW1") (unit 1) (value "SW_SPDT") (footprint "Button_Switch_THT:SW_E-Switch_EG1224_SPDT_Angled")
     )
     (path "/e9d5a963-11d4-45db-b454-4273fc521541"
-      (reference "V1") (unit 1) (value "9V") (footprint "")
+      (reference "V1") (unit 1) (value "9V") (footprint "Connector_JST:JST_PH_B2B-PH-K_1x02_P2.00mm_Vertical")
     )
   )
